File: hardware/keyboard.kicad_pcb (KiCad board)
At the start: 2 copper layers, 140 parts, among them J1 USB_OTG, U1 ATMEGA32U4-AU, U2 MCP23018_SSOP, Y1 16MHz

Commit message: Add HWB, breakouts, LED to sch
Parts:
- added D66: LED, LEDs:LED_1206, F.Cu at (45.3, 11.6)
- added D99: LED, LEDs:LED_1206, F.Cu at (51.2, 5.83)
- added J10: PD5, Connectors:1pin, F.Cu at (3.13, 18.4)
- added J11: PD6, Connectors:1pin, F.Cu at (20.3, 1.48)
- added J12: PD7, Connectors:1pin, F.Cu at (14.7, 9.57)
- added J13: PE6, Connectors:1pin, F.Cu at (0.65, 26.5)
- added J14: PF0, Connectors:1pin, F.Cu at (26.0, 1.48)
- added J15: PF1, Connectors:1pin, F.Cu at (8.78, 11.7)
- added J16: PF4, Connectors:1pin, F.Cu at (20.3, 9.57)
- added J17: PF5, Connectors:1pin, F.Cu at (31.6, 1.48)
- added J18: PF6, Connectors:1pin, F.Cu at (8.78, 19.8)
- added J19: PF7, Connectors:1pin, F.Cu at (14.4, 17.7)
- added J2: PB5, Connectors:1pin, F.Cu at (31.6, 9.57)
- added J3: PB6, Connectors:1pin, F.Cu at (37.3, 1.48)
- added J4: PB7, Connectors:1pin, F.Cu at (14.4, 25.8)
- added J5: PC6, Connectors:1pin, F.Cu at (6.30, 27.9)
- added J6: PC7, Connectors:1pin, F.Cu at (20.1, 17.7)
- added J7: PD2, Connectors:1pin, F.Cu at (26.0, 9.57)
- added J8: PD3, Connectors:1pin, F.Cu at (14.7, 1.48)
- added J9: PD4, Connectors:1pin, F.Cu at (25.7, 17.7)
- added R4: 1k, Resistors_SMD:R_1206_HandSoldering, F.Cu at (32.0, 16.5)
- added R5: 1k, Resistors_SMD:R_1206_HandSoldering, F.Cu at (50.5, 0.28)
- added R6: 2k2, Resistors_SMD:R_1206_HandSoldering, F.Cu at (20.7, 30.4)
- added R7: 2k2, Resistors_SMD:R_1206_HandSoldering, F.Cu at (27.7, 24.6)
- added R8: 1k, Resistors_SMD:R_1206_HandSoldering, F.Cu at (44.9, 6.08)
- added S99: SPST, Buttons_Switches_SMD:SW_SPST_EVQP0, F.Cu at (7.15, 2.33)
- D1: value LED -> D_Small; footprint LEDs:LED_1206 -> Diodes_SMD:D_1206
- D65: value D_Small -> LED; footprint Diodes_SMD:D_1206 -> LEDs:LED_1206
- moved D32 349.0 mm to (51.7, 162.4)
- moved Y1 346.4 mm to (50.9, 11.8)
- moved D46 319.7 mm to (11.1, 65.8)
- moved D40 313.9 mm to (11.1, 114.1)
- moved D47 313.6 mm to (11.1, 41.7)
- moved D62 300.8 mm to (11.1, 186.5)
- moved S40 296.9 mm to (-1.76, 121.0)
- moved S46 294.9 mm to (-1.76, 72.7)
- moved D39 293.5 mm to (51.7, 90.0)
- moved S32 289.9 mm to (38.8, 169.3)
- moved D52 289.6 mm to (51.7, 186.5)
- moved D45 286.7 mm to (51.7, 41.7)
- moved D64 281.8 mm to (11.1, 162.4)
- moved D1 277.6 mm to (132.8, 120.9)
- moved U1 277.2 mm to (-4.50, 5.88)
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Connections:
- net /K10/ROW renamed /KEYS/sheet594A0CEB/ROW
- net /SCL renamed SCL
- net /SDA renamed SDA
- D1 pad 1: GND -> COL0
- D11 pad 1: COL1 -> COL2
- D16 pad 1: COL2 -> COL3
- D21 pad 1: COL3 -> COL4
- D26 pad 1: COL4 -> COL5
- D31 pad 1: COL5 -> COL6
- D36 pad 1: COL6 -> COL7
- D4 pad 1: COL0 -> (no net)
- D41 pad 1: COL7 -> COL8
- D46 pad 1: COL8 -> COL9
- D51 pad 1: COL9 -> COL10
- D56 pad 1: COL10 -> COL11
- D6 pad 1: COL0 -> COL1
- D61 pad 1: COL11 -> COL12
- D65 pad 1: COL12 -> GND
- R3 pad 2: Net-(D1-Pad2) -> Net-(D99-Pad2)
- S1 pad 2: Net-(D2-Pad2) -> Net-(D1-Pad2)
- S10 pad 2: Net-(D11-Pad2) -> Net-(D10-Pad2)
- S11 pad 2: Net-(D12-Pad2) -> Net-(D11-Pad2)
- S12 pad 2: Net-(D13-Pad2) -> Net-(D12-Pad2)
- S13 pad 2: Net-(D14-Pad2) -> Net-(D13-Pad2)
- S14 pad 2: Net-(D15-Pad2) -> Net-(D14-Pad2)
- S15 pad 2: Net-(D16-Pad2) -> Net-(D15-Pad2)
- S16 pad 2: Net-(D17-Pad2) -> Net-(D16-Pad2)
- S17 pad 2: Net-(D18-Pad2) -> Net-(D17-Pad2)
- S18 pad 2: Net-(D19-Pad2) -> Net-(D18-Pad2)
- S19 pad 2: Net-(D20-Pad2) -> Net-(D19-Pad2)
- S2 pad 2: Net-(D3-Pad2) -> Net-(D2-Pad2)
- S20 pad 2: Net-(D21-Pad2) -> Net-(D20-Pad2)
- S21 pad 2: Net-(D22-Pad2) -> Net-(D21-Pad2)
- S22 pad 2: Net-(D23-Pad2) -> Net-(D22-Pad2)
- S23 pad 2: Net-(D24-Pad2) -> Net-(D23-Pad2)
- S24 pad 2: Net-(D25-Pad2) -> Net-(D24-Pad2)
- S25 pad 2: Net-(D26-Pad2) -> Net-(D25-Pad2)
- S26 pad 2: Net-(D27-Pad2) -> Net-(D26-Pad2)
- S27 pad 2: Net-(D28-Pad2) -> Net-(D27-Pad2)
- S28 pad 2: Net-(D29-Pad2) -> Net-(D28-Pad2)
- S29 pad 2: Net-(D30-Pad2) -> Net-(D29-Pad2)
- S3 pad 2: Net-(D4-Pad2) -> Net-(D3-Pad2)
- S30 pad 2: Net-(D31-Pad2) -> Net-(D30-Pad2)
- S31 pad 2: Net-(D32-Pad2) -> Net-(D31-Pad2)
- S32 pad 2: Net-(D33-Pad2) -> Net-(D32-Pad2)
- S33 pad 2: Net-(D34-Pad2) -> Net-(D33-Pad2)
- S34 pad 2: Net-(D35-Pad2) -> Net-(D34-Pad2)
- S35 pad 2: Net-(D36-Pad2) -> Net-(D35-Pad2)
- S36 pad 2: Net-(D37-Pad2) -> Net-(D36-Pad2)
- S37 pad 2: Net-(D38-Pad2) -> Net-(D37-Pad2)
- S38 pad 2: Net-(D39-Pad2) -> Net-(D38-Pad2)
- S39 pad 2: Net-(D40-Pad2) -> Net-(D39-Pad2)
- S4 pad 1: ROW3 -> (no net)
- S4 pad 2: Net-(D5-Pad2) -> Net-(D4-Pad2)
- S40 pad 2: Net-(D41-Pad2) -> Net-(D40-Pad2)
- S41 pad 2: Net-(D42-Pad2) -> Net-(D41-Pad2)
- S42 pad 2: Net-(D43-Pad2) -> Net-(D42-Pad2)
- S43 pad 2: Net-(D44-Pad2) -> Net-(D43-Pad2)
- S44 pad 2: Net-(D45-Pad2) -> Net-(D44-Pad2)
- S45 pad 2: Net-(D46-Pad2) -> Net-(D45-Pad2)
- S46 pad 2: Net-(D47-Pad2) -> Net-(D46-Pad2)
- S47 pad 2: Net-(D48-Pad2) -> Net-(D47-Pad2)
- S48 pad 2: Net-(D49-Pad2) -> Net-(D48-Pad2)
- S49 pad 2: Net-(D50-Pad2) -> Net-(D49-Pad2)
- S5 pad 2: Net-(D6-Pad2) -> Net-(D5-Pad2)
- S50 pad 2: Net-(D51-Pad2) -> Net-(D50-Pad2)
- S51 pad 2: Net-(D52-Pad2) -> Net-(D51-Pad2)
- S52 pad 2: Net-(D53-Pad2) -> Net-(D52-Pad2)
- S53 pad 2: Net-(D54-Pad2) -> Net-(D53-Pad2)
- S54 pad 2: Net-(D55-Pad2) -> Net-(D54-Pad2)
- S55 pad 2: Net-(D56-Pad2) -> Net-(D55-Pad2)
- S56 pad 2: Net-(D57-Pad2) -> Net-(D56-Pad2)
- S57 pad 2: Net-(D58-Pad2) -> Net-(D57-Pad2)
- S58 pad 2: Net-(D59-Pad2) -> Net-(D58-Pad2)
- S59 pad 2: Net-(D60-Pad2) -> Net-(D59-Pad2)
- S6 pad 2: Net-(D7-Pad2) -> Net-(D6-Pad2)
- S60 pad 2: Net-(D61-Pad2) -> Net-(D60-Pad2)
- S61 pad 2: Net-(D62-Pad2) -> Net-(D61-Pad2)
- S62 pad 2: Net-(D63-Pad2) -> Net-(D62-Pad2)
- S63 pad 2: Net-(D64-Pad2) -> Net-(D63-Pad2)
- S64 pad 2: Net-(D65-Pad2) -> Net-(D64-Pad2)
- S7 pad 2: Net-(D8-Pad2) -> Net-(D7-Pad2)
- S8 pad 2: Net-(D9-Pad2) -> Net-(D8-Pad2)
- S9 pad 2: Net-(D10-Pad2) -> Net-(D9-Pad2)
- U1 pad 1: (no net) -> /PE6
- U1 pad 12: (no net) -> /PB7
- U1 pad 13: (no net) -> Net-(S99-Pad2)
- U1 pad 20: (no net) -> /PD2
- U1 pad 21: (no net) -> /PD3
- U1 pad 22: (no net) -> /PD5
- U1 pad 25: (no net) -> /PD4
- U1 pad 26: (no net) -> /PD6
- U1 pad 27: (no net) -> /PD7
- U1 pad 29: (no net) -> /PB5
- U1 pad 30: (no net) -> /PB6
- U1 pad 31: (no net) -> /PC6
- U1 pad 32: (no net) -> /PC7
- U1 pad 33: (no net) -> Net-(R8-Pad2)
- U1 pad 36: (no net) -> /PF7
- U1 pad 37: (no net) -> /PF6
- U1 pad 38: (no net) -> /PF5
- U1 pad 39: (no net) -> /PF4
- U1 pad 40: (no net) -> /PF1
- U1 pad 41: (no net) -> /PF0

Commit message: Move diodes in script, add big thumb buttons
Parts:
- added D100, D101, D102: LED, LEDs:LED_1206, F.Cu at (0.00, 0.00)
- added S100: SPST, Buttons_Switches_SMD:SW_SPST_EVQP0, F.Cu at (0.00, 0.00)
- R1, R2: value 22 -> 1k
- R4, R5: value 1k -> 2k2
- R6, R7: value 2k2 -> 22
- S61, S62, S63, S64: footprint keyboard-modules:CHERRY_PCB_100H -> keyboard-modules:CHERRY_PCB_150H
- moved D3 248.7 mm to (80.1, 140.7), turned to 170 degrees
- moved S3 236.0 mm to (82.1, 146.7), turned to 350 degrees
- moved D11 226.6 mm to (125.0, 105.0), turned to 170 degrees
- moved D14 226.0 mm to (115.1, 161.1), turned to 170 degrees
- moved S14 213.8 mm to (117.1, 167.1), turned to 350 degrees
- moved S11 213.0 mm to (127.0, 111.0), turned to 350 degrees
- moved S62 209.1 mm to (207.0, 204.3), turned to 80 degrees
- moved D23 206.0 mm to (155.8, 149.0), turned to 170 degrees
- moved D62 194.3 mm to (205.0, 198.3), turned to 260 degrees
- moved D21 194.0 mm to (162.4, 111.6), turned to 170 degrees
- moved S23 192.7 mm to (157.8, 155.0), turned to 350 degrees
- moved D28 181.5 mm to (174.0, 155.2), turned to 170 degrees
- moved D8 181.3 mm to (99.2, 142.1), turned to 170 degrees
- moved S21 180.4 mm to (164.4, 117.6), turned to 350 degrees
- moved D15 178.5 mm to (111.8, 179.8), turned to 170 degrees
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Connections:
- net /KEYS/sheet594A0CEB/ROW renamed /KEYS/KCEB/ROW
- D4 pad 1: (no net) -> COL0
- D65 pad 2: Net-(D65-Pad2) -> (no net)
- D66 pad 2: Net-(D66-Pad2) -> (no net)
- D99 pad 2: Net-(D99-Pad2) -> (no net)
- R1 pad 1: Net-(R1-Pad1) -> +5V
- R1 pad 2: Net-(J1-Pad3) -> Net-(D100-Pad2)
- R2 pad 1: Net-(R2-Pad1) -> (no net)
- R2 pad 2: Net-(J1-Pad2) -> Net-(D101-Pad2)
- R3 pad 1: +5V -> (no net)
- R3 pad 2: Net-(D99-Pad2) -> Net-(D102-Pad2)
- R4 pad 1: (no net) -> +5V
- R4 pad 2: Net-(D65-Pad2) -> SCL
- R5 pad 1: (no net) -> +5V
- R5 pad 2: Net-(D66-Pad2) -> SDA
- R6 pad 1: +5V -> Net-(R6-Pad1)
- R6 pad 2: SCL -> Net-(J1-Pad3)
- R7 pad 1: +5V -> Net-(R7-Pad1)
- R7 pad 2: SDA -> Net-(J1-Pad2)
- S4 pad 1: (no net) -> ROW3
- U1 pad 13: Net-(S99-Pad2) -> Net-(S100-Pad2)
- U1 pad 3: Net-(R2-Pad1) -> Net-(R7-Pad1)
- U1 pad 4: Net-(R1-Pad1) -> Net-(R6-Pad1)

Commit message: Start layout of right hand
Parts:
- moved S47 328.2 mm to (316.3, 129.7), turned to 10 degrees
- moved S60 328.0 mm to (364.5, 184.1), turned to 10 degrees
- moved S46 317.1 mm to (313.0, 111.0), turned to 10 degrees
- moved D47 314.1 mm to (314.3, 123.7), turned to 190 degrees
- moved S44 313.5 mm to (303.7, 167.5), turned to 10 degrees
- moved D60 313.4 mm to (362.5, 178.1), turned to 190 degrees
- moved S52 303.6 mm to (335.5, 129.3), turned to 10 degrees
- moved D46 302.4 mm to (311.0, 105.0), turned to 190 degrees
- moved S45 301.4 mm to (307.0, 186.2), turned to 10 degrees
- moved D44 299.2 mm to (301.7, 161.5), turned to 190 degrees
- moved S40 299.2 mm to (288.8, 192.4), turned to 10 degrees
- moved D52 288.8 mm to (333.5, 123.3), turned to 190 degrees
- moved D45 288.7 mm to (305.0, 180.2), turned to 190 degrees
- moved S48 287.1 mm to (319.6, 148.4), turned to 10 degrees
- moved D40 285.0 mm to (286.8, 186.4), turned to 190 degrees
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
Commit message: Don't flip diodes if already on B.Cu
Parts:
- removed D65, D66, D99: LED, LEDs:LED_1206
- removed S99: SPST, Buttons_Switches_SMD:SW_SPST_EVQP0
- D1, D10, D11, D12, D13, D14, D15, D16, D17, D18, D19, D2, D20, D21, D22, D23, D24, D25, D26, D27, D28, D29, D3, D30, D31, D32, D33, D34, D35, D36, D37, D38, D39, D4, D40, D41, D42, D43, D44, D45, D46, D47, D48, D49, D5, D50, D51, D52, D53, D54, D55, D56, D57, D58, D59, D6, D60, D61, D62, D63, D64, D7, D8, D9: moved to B.Cu
- moved R5 120.1 mm to (148.5, 105.0)
- moved Y1 115.0 mm to (148.5, 105.0)
- moved C3 114.2 mm to (148.5, 105.0)
- moved R8 112.3 mm to (148.5, 105.0)
- moved J3 108.2 mm to (148.5, 105.0)
- moved C2 105.2 mm to (148.5, 105.0)
- moved J17 103.5 mm to (148.5, 105.0)
- moved R3 103.3 mm to (148.5, 105.0)
- moved U2 99.9 mm to (148.5, 105.0)
- moved J2 99.1 mm to (148.5, 105.0)
- moved J14 99.0 mm to (148.5, 105.0)
- moved R4 96.1 mm to (148.5, 105.0)
- moved J11 94.5 mm to (148.5, 105.0)
- moved J7 94.3 mm to (148.5, 105.0)
- moved J8 90.2 mm to (148.5, 105.0)
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Other:
- rule pad_to_mask_clearance: 0.2 -> 0

Commit message: Replace 1.5u with 2u thumb keys
Parts:
- S61, S62, S63, S64: footprint keyboard-modules:CHERRY_PCB_150H -> keyboard-modules:CHERRY_PCB_200V
- moved D60 7.99 mm to (325.5, 112.4)
- moved S60 7.99 mm to (327.5, 118.4)
- moved D59 7.98 mm to (322.2, 93.6)
- moved S59 7.98 mm to (324.2, 99.6)
- moved D58 7.97 mm to (318.9, 74.8)
- moved S58 7.97 mm to (320.9, 80.8)
- moved D57 7.96 mm to (315.5, 56.1)
- moved S57 7.96 mm to (317.5, 62.1)
- moved D56 7.95 mm to (312.2, 37.3)
- moved S56 7.95 mm to (314.2, 43.3)
- moved D55 7.94 mm to (306.4, 113.7)
- moved S55 7.94 mm to (308.4, 119.7)
- moved D54 7.93 mm to (303.1, 94.9)
- moved S54 7.93 mm to (305.1, 100.9)
- moved D53 7.92 mm to (299.7, 76.2)
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