File: hardware/keyboard.kicad_pcb (KiCad board)
At the start: 2 copper layers, 321.6 x 127.7 mm, 154 parts, among them J1 USB_OTG, U1 ATMEGA32U4-AU, U2 MCP23018_SSOP, Y1 16MHz

Commit message: WIP for V2 fixes
Parts:
- removed G***: LOGO, matt:hbnum2-small
- removed REF** (x5): MountingHole_3.2mm_M3, MountingHole_3.2mm_M3
- added J10: CONN_01X01, keyboard-modules:CONN_1, F.Cu at (179.5, 72.2)
- added J11: CONN_01X01, keyboard-modules:CONN_1, F.Cu at (180.6, 72.6)
- added J12: CONN_01X01, keyboard-modules:CONN_1, F.Cu at (182.2, 72.4)
- added J13: CONN_01X01, keyboard-modules:CONN_1, F.Cu at (183.4, 72.9)
- added J14: CONN_01X01, keyboard-modules:CONN_1, F.Cu at (185.1, 73.0)
- added J2: CONN_01X01, keyboard-modules:CONN_1, F.Cu at (183.6, 87.9)
- added J3: CONN_01X01, keyboard-modules:CONN_1, F.Cu at (184.9, 87.8)
- added J4: CONN_01X01, keyboard-modules:CONN_1, F.Cu at (189.5, 82.8)
- added J5: CONN_01X01, keyboard-modules:CONN_1, F.Cu at (186.2, 87.8)
- added J6: CONN_01X01, keyboard-modules:CONN_1, F.Cu at (189.3, 81.8)
- added J7: CONN_01X01, keyboard-modules:CONN_1, F.Cu at (189.6, 80.5)
- added J8: CONN_01X01, keyboard-modules:CONN_1, F.Cu at (173.4, 75.0)
- added J9: CONN_01X01, keyboard-modules:CONN_1, F.Cu at (177.8, 72.1)
- J1: footprint Connectors_USB:USB_Micro-B_Molex-105017-0001 -> keyboard-modules:USB-MINI
- U2: footprint Housings_SSOP:SSOP-28_5.3x10.2mm_Pitch0.65mm -> Housings_SSOP:SSOP-24_5.3x8.2mm_Pitch0.65mm
- Y1: footprint Crystals:Crystal_SMD_3225-4pin_3.2x2.5mm_HandSoldering -> Crystals:Crystal_Round_d1.0mm_Vertical
- moved R6 3.89 mm to (176.4, 45.0)
- moved R7 3.89 mm to (179.0, 45.0)
- moved F1 3.89 mm to (182.0, 45.0)
- moved C1 1.15 mm to (181.7, 90.4)
- moved Y1 1.13 mm to (179.7, 88.7)
- moved C2 0.94 mm to (176.1, 90.6)
- moved U2 0.69 mm to (178.8, 108.3)
- moved J1 0.27 mm to (179.3, 34.2), turned to 270 degrees
- moved S100 0.26 mm to (168.8, 38.4)
Connections:
- U1 pad 14: VCC -> +5V
- U1 pad 24: VCC -> +5V
- U1 pad 31: /PC6 -> (no net)
- U1 pad 32: /PC7 -> (no net)
- U1 pad 34: VCC -> +5V
- U1 pad 44: VCC -> +5V
Routing:
- net COL11: track 226.3 -> 80.9 mm, vias 1 -> 0
- net COL10: track 207.0 -> 81.2 mm, vias 1 -> 0
- net COL12: track 110.5 -> 61.9 mm, vias 3 -> 2
- net VCC: track 30.5 -> 0.00 mm, vias 4 -> 0
- net +5V: track 107.8 -> 126.9 mm, vias 9 -> 11
- net Net-(R8-Pad2): track 7.48 -> 2.71 mm, vias 1 -> 0
- net COL6: track 126.5 -> 130.6 mm
- net COL7: track 143.8 -> 145.1 mm
- net COL9: track 185.7 -> 184.9 mm
- net COL8: track 166.0 -> 165.2 mm
- removed copper zone on B.Cu, net GND
- removed copper zone on F.Cu, net GND

Commit message: More WIP on V2
Parts:
- F1: footprint Fuse_Holders_and_Fuses:Fuse_SMD1206_HandSoldering -> Resistors_SMD:R_1206_HandSoldering
- moved J14 2.92 mm to (182.2, 72.2)
- moved C1 2.61 mm to (181.5, 93.0)
- moved J7 2.59 mm to (187.0, 80.8)
- moved J4 2.50 mm to (187.0, 83.2)
- moved C2 2.42 mm to (176.5, 93.0)
- moved J6 2.29 mm to (187.0, 82.0)
- moved J13 2.19 mm to (181.2, 73.2)
- moved J5 1.67 mm to (184.5, 87.8)
- moved J12 1.66 mm to (180.5, 72.2)
- moved J2 1.63 mm to (182.0, 87.8)
- moved J3 1.63 mm to (183.2, 87.8)
- moved R8 1.55 mm to (189.0, 79.0)
- moved J11 1.26 mm to (179.5, 73.2)
- moved J9 1.23 mm to (177.5, 73.2)
- moved J10 0.98 mm to (178.5, 72.2)
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Connections:
- J1 pad 4: (no net) -> Net-(J1-Pad4)
- U1 pad 28: (no net) -> ROW4
- U1 pad 31: (no net) -> /PC6
- U1 pad 32: (no net) -> /PC7
- U1 pad 42: (no net) -> Net-(U1-Pad42)
- U2 pad 13: (no net) -> Net-(U2-Pad13)
- U2 pad 14: (no net) -> Net-(U2-Pad14)
- U2 pad 15: (no net) -> Net-(U2-Pad15)
- U2 pad 16: (no net) -> Net-(U2-Pad16)
- U2 pad 24: (no net) -> Net-(U2-Pad24)
- U2 pad 8: (no net) -> Net-(U2-Pad8)
- U2 pad 9: (no net) -> Net-(U2-Pad9)
Routing:
- net GND: track 177.9 -> 0.00 mm, vias 9 -> 0
- net Net-(J1-Pad6): track 19.4 -> 0.00 mm
- net Net-(J1-Pad3): track 4.46 -> 0.15 mm
- net Net-(F1-Pad2): track 3.85 -> 0.00 mm
- net /PF7: track 0.00 -> 2.59 mm
- net /PF5: track 0.00 -> 2.52 mm
- net /PF1: track 0.00 -> 2.49 mm
- net Net-(J1-Pad2): track 2.91 -> 0.73 mm
- net /PD5: track 0.00 -> 2.10 mm
- net /PD4: track 0.00 -> 2.03 mm
- net /PD7: track 0.00 -> 2.01 mm
- net /PD3: track 0.00 -> 1.92 mm
- net /PD6: track 0.00 -> 1.85 mm
- net /PE6: track 0.00 -> 1.74 mm
- net /PD2: track 0.00 -> 1.73 mm
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
Commit message: Add more mounting holes, re-route updated components
Parts:
- removed D101: LED_RGB, LEDs:LED_RGB_PLCC-6
- removed J10, J11, J12, J13, J14, J2, J3, J4, J5, J6, J7, J8, J9: CONN_01X01, keyboard-modules:CONN_1
- removed R1, R3: 1k, Resistors_SMD:R_1206_HandSoldering
- added D65: LED_CRGB, LEDs:LED_D5.0mm-4, F.Cu at (190.8, 80.3)
- added GND: CONN_01X01, keyboard-modules:CONN_1, F.Cu at (174.0, 38.9)
- added PB7: CONN_01X01, keyboard-modules:CONN_1, F.Cu at (173.2, 89.7)
- added PD2: CONN_01X01, keyboard-modules:CONN_1, F.Cu at (188.0, 89.7)
- added PD3: CONN_01X01, keyboard-modules:CONN_1, F.Cu at (188.0, 93.5)
- added PD4: CONN_01X01, keyboard-modules:CONN_1, F.Cu at (191.0, 89.7)
- added PD5: CONN_01X01, keyboard-modules:CONN_1, F.Cu at (191.0, 93.5)
- added PD6: CONN_01X01, keyboard-modules:CONN_1, F.Cu at (193.8, 89.7)
- added PE6: CONN_01X01, keyboard-modules:CONN_1, F.Cu at (171.2, 74.4)
- added PF0: CONN_01X01, keyboard-modules:CONN_1, F.Cu at (173.5, 69.8)
- added PF1: CONN_01X01, keyboard-modules:CONN_1, F.Cu at (170.9, 68.1)
- added PF4: CONN_01X01, keyboard-modules:CONN_1, F.Cu at (173.5, 66.3)
- added PF5: CONN_01X01, keyboard-modules:CONN_1, F.Cu at (185.9, 66.3)
- added PF6: CONN_01X01, keyboard-modules:CONN_1, F.Cu at (188.5, 68.1)
- added PF7: CONN_01X01, keyboard-modules:CONN_1, F.Cu at (185.9, 69.8)
- added REF**: MountingHole_3.2mm_M3, MountingHole_3.2mm_M3, F.Cu at (230.9, 148.9)
- added REF**: MountingHole_3.2mm_M3, MountingHole_3.2mm_M3, F.Cu at (127.1, 148.9)
- added REF**: MountingHole_3.2mm_M3, MountingHole_3.2mm_M3, F.Cu at (179.0, 155.9)
- added REF**: MountingHole_3.2mm_M3, MountingHole_3.2mm_M3, F.Cu at (335.5, 130.5)
- added REF**: MountingHole_3.2mm_M3, MountingHole_3.2mm_M3, F.Cu at (22.5, 130.5)
- added REF**: MountingHole_3.2mm_M3, MountingHole_3.2mm_M3, F.Cu at (316.7, 28.9)
- added REF**: MountingHole_3.2mm_M3, MountingHole_3.2mm_M3, F.Cu at (230.7, 28.9)
- added REF**: MountingHole_3.2mm_M3, MountingHole_3.2mm_M3, F.Cu at (127.3, 28.9)
- added REF**: MountingHole_3.2mm_M3, MountingHole_3.2mm_M3, F.Cu at (41.3, 28.9)
- added SCL: CONN_01X01, keyboard-modules:CONN_1, F.Cu at (183.4, 100.3)
- added SDA: CONN_01X01, keyboard-modules:CONN_1, F.Cu at (186.7, 100.3)
- added VCC: CONN_01X01, keyboard-modules:CONN_1, F.Cu at (184.4, 38.9)
- R2: moved to B.Cu
- moved R2 38.8 mm to (192.8, 75.7)
- moved S100 9.50 mm to (168.7, 28.9)
- moved R6 8.17 mm to (176.5, 36.8)
- moved R7 8.14 mm to (179.1, 36.9)
- moved F1 8.14 mm to (181.6, 36.9)
- moved J1 7.52 mm to (179.1, 26.7)
- moved R8 5.00 mm to (192.8, 75.7), turned to 180 degrees
Connections:
- J1 pad 4: Net-(J1-Pad4) -> (no net)
- U1 pad 12: LED3 -> Net-(PB7-Pad1)
- U1 pad 27: /PD7 -> LED3
- U1 pad 28: ROW4 -> (no net)
- U1 pad 31: /PC6 -> (no net)
- U1 pad 32: /PC7 -> (no net)
- U1 pad 42: Net-(U1-Pad42) -> (no net)
- U2 pad 13: Net-(U2-Pad13) -> (no net)
- U2 pad 14: Net-(U2-Pad14) -> (no net)
- U2 pad 15: Net-(U2-Pad15) -> (no net)
- U2 pad 16: Net-(U2-Pad16) -> (no net)
- U2 pad 24: Net-(U2-Pad24) -> (no net)
- U2 pad 8: Net-(U2-Pad8) -> (no net)
- U2 pad 9: Net-(U2-Pad9) -> (no net)
Routing:
- net COL11: track 80.9 -> 223.7 mm, vias 0 -> 1
- net COL10: track 81.2 -> 204.9 mm, vias 0 -> 1
- net LED3: track 69.3 -> 10.2 mm, vias 2 -> 0
- net COL12: track 61.9 -> 102.3 mm, vias 2 -> 4
- net LED1: track 46.6 -> 7.85 mm, vias 2 -> 0
- net LED2: track 47.0 -> 9.32 mm, vias 2 -> 0
- net +5V: track 126.9 -> 141.4 mm
- net /PD6: track 1.85 -> 16.1 mm, vias 0 -> 1
- net /PF4: track 1.44 -> 14.5 mm, vias 0 -> 2
- net /PF6: track 1.50 -> 14.0 mm, vias 0 -> 2
- net /PD5: track 2.10 -> 14.5 mm, vias 0 -> 2
- net /PF1: track 2.49 -> 14.3 mm, vias 0 -> 2
- net /PF5: track 2.52 -> 14.0 mm, vias 0 -> 2
- net /PD4: track 2.03 -> 12.7 mm, vias 0 -> 1
- net /PD3: track 1.92 -> 12.6 mm, vias 0 -> 2
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Other:
- board size 321.6 x 127.7 mm -> 321.6 x 135 mm

Commit message: Add ground fills
Routing:
- net GND: track 0.00 -> 51.6 mm
- added copper zone on B.Cu, net GND
- added copper zone on F.Cu, net GND
Changed lines of the file:
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@@
   (general
     (links 256)
-    (no_connects 16)
+    (no_connects 0)
     (area 13.09439 23.434285 344.905608 190.075001)
     (thickness 1.6)
     (drawings 8)
-    (tracks 776)
+    (tracks 804)
     (zones 0)
     (modules 172)
@@
     (pad_to_mask_clearance 0)
     (aux_axis_origin 0 0)
-    (visible_elements FFFFFF7F)
+    (visible_elements FFFFEF7F)
     (pcbplotparams
       (layerselection 0x010f0_ffffffff)
@@
   (gr_line (start 179 40) (end 179 190) (layer Dwgs.User) (width 0.15))
   (gr_line (start 179 40) (end 179 190) (layer Dwgs.User) (width 0.15))
+  (segment (start 182.664 73.368) (end 183.134 72.898) (width 0.25) (layer F.Cu) (net 1))
+  (segment (start 182.664 74.676) (end 182.664 73.368) (width 0.25) (layer F.Cu) (net 1))
+  (segment (start 194.754 73.342) (end 194.564 73.152) (width 0.25) (layer F.Cu) (net 1))
+  (segment (start 194.754 75.692) (end 194.754 73.342) (width 0.25) (layer F.Cu) (net 1))
+  (segment (start 178.737 84.074) (end 183.862 84.074) (width 0.25) (layer F.Cu) (net 1))
+  (segment (start 183.862 84.074) (end 184.164 84.376) (width 0.25) (layer F.Cu) (net 1))
+  (segment (start 184.164 84.376) (end 185.164 84.376) (width 0.25) (layer F.Cu) (net 1))
+  (segment (start 173.764 79.576) (end 174.239 79.576) (width 0.25) (layer F.Cu) (net 1))
+  (segment (start 174.239 79.576) (end 178.737 84.074) (width 0.25) (layer F.Cu) (net 1))
+  (segment (start 177.8 87.14) (end 177.8 87.376) (width 0.25) (layer F.Cu) (net 1))
+  (segment (start 177.864 86.076) (end 177.864 87.076) (width 0.25) (layer F.Cu) (net 1))
+  (segment (start 177.864 87.076) (end 177.8 87.14) (width 0.25) (layer F.Cu) (net 1))
+  (segment (start 176.948 110.58) (end 181.07 106.458) (width 0.25) (layer F.Cu) (net 1))
+  (segment (start 181.07 106.458) (end 181.07 102.362) (width 0.25) (layer F.Cu) (net 1))
+  (segment (start 175.21 110.58) (end 176.948 110.58) (width 0.25) (layer F.Cu) (net 1))
+  (segment (start 170.686 72.39) (end 167.418 75.658) (width 0.25) (layer F.Cu) (net 1))
+  (segment (start 167.418 75.658) (end 167.418 77.216) (width 0.25) (layer F.Cu) (net 1))
+  (segment (start 172.466 72.644) (end 170.94 72.644) (width 0.25) (layer F.Cu) (net 1))
+  (segment (start 170.94 72.644) (end 170.686 72.39) (width 0.25) (layer F.Cu) (net 1))
+  (segment (start 172.974 73.152) (end 172.466 72.644) (width 0.25) (layer F.Cu) (net 1))
+  (segment (start 175.74 73.152) (end 172.974 73.152) (width 0.25) (layer F.Cu) (net 1))
+  (segment (start 176.264 74.676) (end 176.264 73.676) (width 0.25) (layer F.Cu) (net 1))
+  (segment (start 176.264 73.676) (end 175.74 73.152) (width 0.25) (layer F.Cu) (net 1))
+  (segment (start 172.453 78.74) (end 170.319 78.74) (width 0.25) (layer F.Cu) (net 1))
+  (segment (start 170.319 78.74) (end 168.668 80.391) (width 0.25) (layer F.Cu) (net 1))
+  (segment (start 168.668 80.391) (end 167.418 80.391) (width 0.25) (layer F.Cu) (net 1))
+  (segment (start 173.764 79.576) (end 173.289 79.576) (width 0.25) (layer F.Cu) (net 1))
+  (segment (start 173.289 79.576) (end 172.453 78.74) (width 0.25) (layer F.Cu) (net 1))
   (segment (start 181.5 91) (end 181.5 90.8) (width 0.25) (layer F.Cu) (net 2) (status 30))
   (segment (start 181.5 90.8) (end 179.75 89.05) (width 0.25) (layer F.Cu) (net 2) (status 30))
@@
   (segment (start 175.464 86.076) (end 175.464 87.426) (width 0.25) (layer F.Cu) (net 114) (status 10))
   (segment (start 175.464 87.426) (end 173.228 89.662) (width 0.25) (layer F.Cu) (net 114) (status 20))
+  (zone (net 1) (net_name GND) (layer F.Cu) (hatch edge 0.508)
+    (connect_pads (clearance 0.508))
+    (min_thickness 0.254)
+    (fill yes (arc_segments 16) (thermal_gap 0.508) (thermal_bridge_width 0.508))
+    (polygon
+      (pts
+        (xy 16.51 23.876) (xy 338.074 21.082) (xy 347.218 141.478) (xy 171.196 169.164) (xy 9.144 132.588)
+        (xy 12.954 37.846)
+      )
+    )
+  )
+  (zone (net 1) (net_name GND) (layer B.Cu) (hatch edge 0.508)
+    (connect_pads (clearance 0.508))
+    (min_thickness 0.254)
+    (fill yes (arc_segments 16) (thermal_gap 0.508) (thermal_bridge_width 0.508))
+    (polygon
+      (pts
+        (xy 23.368 20.32) (xy 331.978 20.828) (xy 347.218 137.668) (xy 170.688 174.244) (xy 0.254 134.62)
+      )
+    )
+  )
 )
