File: hardware/ThumbKey.sch (KiCad schematic (older format))
At the start: 2 parts

Commit message: More routing
Parts:
- D61: footprint Diodes_SMD:D_1206 -> d_mod:D_1206
Changed lines of the file:
@@
 F 0 "D64" H 2350 1880 50  0000 L CNN
 F 1 "D_Small" H 2250 1720 50  0000 L CNN
-F 2 "Diodes_SMD:D_1206" V 2400 1800 50  0001 C CNN
+F 2 "d_mod:D_1206" V 2400 1800 50  0001 C CNN
 F 3 "" V 2400 1800 50  0001 C CNN
 	1    2400 1800

Commit message: Update parts after starting sourcing
Parts:
- D61: footprint d_mod:D_1206 -> Diodes_SMD:D_SOD-123
Changed lines of the file:
@@
 F 0 "D64" H 2350 1880 50  0000 L CNN
 F 1 "D_Small" H 2250 1720 50  0000 L CNN
-F 2 "d_mod:D_1206" V 2400 1800 50  0001 C CNN
+F 2 "Diodes_SMD:D_SOD-123" V 2400 1800 50  0001 C CNN
 F 3 "" V 2400 1800 50  0001 C CNN
 	1    2400 1800
