File: hardware/Key.sch (KiCad schematic (older format))
At the start: 2 parts

Commit message: WIP for V2 fixes
Changed lines of the file:
@@
 LIBS:valves
 LIBS:keyboard-cache
-EELAYER 26 0
+EELAYER 25 0
 EELAYER END
 $Descr A4 11693 8268
@@
 AR Path="/5947FBED/594A0F7E/5940D01B" Ref="S59"  Part="1"
 AR Path="/5947FBED/594A0F88/5940D01B" Ref="S60"  Part="1"
-F 0 "S1" H 2600 1600 60  0000 R CNN
+F 0 "S60" H 2600 1600 60  0000 R CNN
 F 1 "SPST" H 2200 1600 60  0000 C CNN
 F 2 "keyboard-modules:CHERRY_PCB_100H" H 2350 1750 60  0001 C CNN
@@
 AR Path="/5947FBED/594A0F7E/5940D05E" Ref="D59"  Part="1"
 AR Path="/5947FBED/594A0F88/5940D05E" Ref="D60"  Part="1"
-F 0 "D1" H 2300 1980 50  0000 L CNN
+F 0 "D60" H 2300 1980 50  0000 L CNN
 F 1 "D_Small" H 2200 1820 50  0000 L CNN
 F 2 "Diodes_SMD:D_SOD-123" V 2350 1900 50  0001 C CNN
